File: template/template.sch (KiCad schematic (older format))
At the start: 0 parts

Commit message: keyboards
Other:
- note added: "Logos / Markings"
Changed lines of the file:
@@
 EESchema Schematic File Version 4
-EELAYER 29 0
+EELAYER 30 0
 EELAYER END
 $Descr A4 11693 8268
 encoding utf-8
 Sheet 1 1
-Title ""
+Title "DESIGN_TITLE"
 Date ""
-Rev "0"
+Rev "VER_NO"
 Comp "Josh Johnson"
 Comment1 ""
@@
 Comment4 ""
 $EndDescr
+$Comp
+L Graphic:Logo_Open_Hardware_Small #LOGO2
+U 1 1 5E2031A4
+P 6600 7500
+F 0 "#LOGO2" H 6600 7886 50  0000 C CNN
+F 1 "OSHW_FMask" H 6600 7795 50  0000 C CNN
+F 2 "josh-logos:OSHW_Logo_3.6x3.6_F.Mask" H 6600 7500 50  0001 C CNN
+F 3 "~" H 6600 7500 50  0001 C CNN
+	1    6600 7500
+	1    0    0    -1
+$EndComp
+$Comp
+L Mechanical:MountingHole #LOGO1
+U 1 1 5E204886
+P 6050 7200
+F 0 "#LOGO1" H 6050 7437 50  0000 C CNN
+F 1 "Josh-Details" H 6050 7346 50  0000 C CNN
+F 2 "josh-logos:josh-details" H 6050 7200 50  0001 C CNN
+F 3 "~" H 6050 7200 50  0001 C CNN
+	1    6050 7200
+	1    0    0    -1
+$EndComp
+$Comp
+L Mechanical:MountingHole #LOGO?
+U 1 1 5E2051A0
+P 6050 7650
+F 0 "#LOGO?" H 6050 7887 50  0000 C CNN
+F 1 "4-Layer-Check" H 6050 7796 50  0000 C CNN
+F 2 "josh-logos:4-layer-check" H 6050 7650 50  0001 C CNN
+F 3 "~" H 6050 7650 50  0001 C CNN
+	1    6050 7650
+	1    0    0    -1
+$EndComp
+Text Notes 5350 6850 0    100  ~ 0
+Logos / Markings
+$Comp
+L Mechanical:MountingHole #LOGO?
+U 1 1 5E2057DD
+P 5400 7650
+F 0 "#LOGO?" H 5400 7887 50  0000 C CNN
+F 1 "Josh-Logo" H 5400 7796 50  0000 C CNN
+F 2 "josh-logos:josh-johnson-logo-8_6x1_5" H 5400 7650 50  0001 C CNN
+F 3 "~" H 5400 7650 50  0001 C CNN
+	1    5400 7650
+	1    0    0    -1
+$EndComp
+$Comp
+L Mechanical:MountingHole #LOGO?
+U 1 1 5E205A57
+P 5400 7200
+F 0 "#LOGO?" H 5400 7437 50  0000 C CNN
+F 1 "Board-Title" H 5400 7346 50  0000 C CNN
+F 2 "josh-logos:board-title" H 5400 7200 50  0001 C CNN
+F 3 "~" H 5400 7200 50  0001 C CNN
+	1    5400 7200
+	1    0    0    -1
+$EndComp
 $EndSCHEMATC

Commit message: updating template
Parts:
- added LOGO1: Josh-Details, josh-logos:josh-details, symbol Mechanical:MountingHole
- added LOGO2: OSHW_FMask, josh-logos:OSHW_Logo_3.6x3.6_F.Mask, symbol Graphic:Logo_Open_Hardware_Small
- added LOGO3: Board-Title, josh-logos:board-title, symbol Mechanical:MountingHole
- added LOGO4: Josh-Logo, josh-logos:josh-johnson-logo-8_6x1_5, symbol Mechanical:MountingHole
- added LOGO5: 4-Layer-Check, josh-logos:4-layer-check, symbol Mechanical:MountingHole
Changed lines of the file:
@@
 $EndDescr
 $Comp
-L Graphic:Logo_Open_Hardware_Small #LOGO2
+L Graphic:Logo_Open_Hardware_Small LOGO2
 U 1 1 5E2031A4
 P 6600 7500
-F 0 "#LOGO2" H 6600 7886 50  0000 C CNN
+F 0 "LOGO2" H 6600 7886 50  0000 C CNN
 F 1 "OSHW_FMask" H 6600 7795 50  0000 C CNN
 F 2 "josh-logos:OSHW_Logo_3.6x3.6_F.Mask" H 6600 7500 50  0001 C CNN
@@
 $EndComp
 $Comp
-L Mechanical:MountingHole #LOGO1
+L Mechanical:MountingHole LOGO1
 U 1 1 5E204886
 P 6050 7200
-F 0 "#LOGO1" H 6050 7437 50  0000 C CNN
+F 0 "LOGO1" H 6050 7437 50  0000 C CNN
 F 1 "Josh-Details" H 6050 7346 50  0000 C CNN
 F 2 "josh-logos:josh-details" H 6050 7200 50  0001 C CNN
@@
 $EndComp
 $Comp
-L Mechanical:MountingHole #LOGO?
+L Mechanical:MountingHole LOGO5
 U 1 1 5E2051A0
 P 6050 7650
-F 0 "#LOGO?" H 6050 7887 50  0000 C CNN
+F 0 "LOGO5" H 6050 7887 50  0000 C CNN
 F 1 "4-Layer-Check" H 6050 7796 50  0000 C CNN
 F 2 "josh-logos:4-layer-check" H 6050 7650 50  0001 C CNN
@@
 Logos / Markings
 $Comp
-L Mechanical:MountingHole #LOGO?
+L Mechanical:MountingHole LOGO4
 U 1 1 5E2057DD
 P 5400 7650
-F 0 "#LOGO?" H 5400 7887 50  0000 C CNN
+F 0 "LOGO4" H 5400 7887 50  0000 C CNN
 F 1 "Josh-Logo" H 5400 7796 50  0000 C CNN
 F 2 "josh-logos:josh-johnson-logo-8_6x1_5" H 5400 7650 50  0001 C CNN
@@
 $EndComp
 $Comp
-L Mechanical:MountingHole #LOGO?
+L Mechanical:MountingHole LOGO3
 U 1 1 5E205A57
 P 5400 7200
-F 0 "#LOGO?" H 5400 7437 50  0000 C CNN
+F 0 "LOGO3" H 5400 7437 50  0000 C CNN
 F 1 "Board-Title" H 5400 7346 50  0000 C CNN
 F 2 "josh-logos:board-title" H 5400 7200 50  0001 C CNN
