File: template/template.kicad_pcb (KiCad board)
At the start: 2 copper layers, 0 parts

Commit message: updating template
Parts:
- added LOGO1: Josh-Details, josh-logos:josh-details, F.Cu at (144.2, 184.9)
- added LOGO2: OSHW_FMask, josh-logos:OSHW_Logo_3.6x3.6_F.Mask, F.Cu at (157.2, 193.9)
- added LOGO3: Board-Title, josh-logos:board-title, F.Cu at (166.8, 184.6)
- added LOGO4: Josh-Logo, josh-logos:josh-johnson-logo-8_6x1_5, F.Cu at (143.1, 193.9)
- added LOGO5: 4-Layer-Check, josh-logos:4-layer-check, F.Cu at (170.9, 194.9)

Commit message: v6 cleanup
Parts:
- removed LOGO1: Josh-Details, josh-logos:josh-details
- removed LOGO3: Board-Title, josh-logos:board-title
- removed LOGO4: Josh-Logo, josh-logos:josh-johnson-logo-8_6x1_5
- removed LOGO5: 4-Layer-Check, josh-logos:4-layer-check
- LOGO2: value OSHW_FMask -> Josh-Details; footprint josh-logos:OSHW_Logo_3.6x3.6_F.Mask -> josh-logos:josh-details; moved to B.Cu
- moved LOGO2 36.3 mm to (192.6, 201.8), turned to 180 degrees
Other:
- net class Default removed

Commit message: bump template to v7
Parts:
- removed LOGO2: Josh-Details, josh-logos:josh-details
Changed lines of the file:
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@@
-(kicad_pcb (version 20210424) (generator pcbnew)
+(kicad_pcb (version 20221018) (generator pcbnew)
   (general
     (thickness 1.6)
@@
     (pcbplotparams
       (layerselection 0x00010fc_ffffffff)
+      (plot_on_all_layers_selection 0x0000000_00000000)
       (disableapertmacros false)
       (usegerberextensions true)
@@
       (usegerberadvancedattributes false)
       (creategerberjobfile false)
-      (svguseinch false)
+      (dashed_line_dash_ratio 12.000000)
+      (dashed_line_gap_ratio 3.000000)
       (svgprecision 6)
-      (excludeedgelayer true)
       (plotframeref false)
       (viasonmask false)
@@
   )
   (net 0 "")
-  (footprint "josh-logos:josh-details" (layer "B.Cu")
-    (at 192.6 201.8 180)
-    (property "DNP" "DNP")
-    (property "Sheetfile" "keyboard.kicad_sch")
-    (property "Sheetname" "")
-    (attr through_hole)
-    (fp_text reference "LOGO2" (at -2.7 2.3) (layer "B.Fab") hide
-      (effects (font (size 1 1) (thickness 0.15)) (justify mirror))
-    )
-    (fp_text value "Josh-Details" (at 0 -3.7) (layer "B.Fab")
-      (effects (font (size 1 1) (thickness 0.15)) (justify mirror))
-    )
-  )
 )
